Commit message: Update ar_macro.xacro

File: annin_ar4_description/urdf/ar_macro.xacro (robot description, xacro)
@@ -2,4 +2,5 @@
 <robot xmlns:xacro="http://wiki.ros.org/xacro">
   <xacro:macro name="ar_robot" params="
+    tf_prefix
     parent
     *origin
@@ -7,10 +8,10 @@
   ">
     <xacro:property name="robot_parameters" value="${xacro.load_yaml(robot_parameters_file)}"/>
-    <joint name="base_joint" type="fixed">
+    <joint name="${tf_prefix}base_joint" type="fixed">
       <xacro:insert_block name="origin" />
       <parent link="${parent}"/>
-      <child link="base_link" />
-    </joint>
-    <link name="base_link">
+      <child link="${tf_prefix}base_link" />
+    </joint>
+    <link name="${tf_prefix}base_link">
       <inertial>
         <origin rpy="0 0 0" xyz="-4.6941E-06 0.054174 0.038824"/>
@@ -34,5 +35,5 @@
       </collision>
     </link>
-    <link name="link_1">
+    <link name="${tf_prefix}link_1">
       <inertial>
         <origin rpy="0 0 0" xyz="-0.022706 0.04294 -0.12205"/>
@@ -56,8 +57,8 @@
       </collision>
     </link>
-    <joint name="joint_1" type="revolute">
+    <joint name="${tf_prefix}joint_1" type="revolute">
       <origin rpy="${pi} 0 0" xyz="0 0 0"/>
-      <parent link="base_link"/>
-      <child link="link_1"/>
+      <parent link="${tf_prefix}base_link"/>
+      <child link="${tf_prefix}link_1"/>
       <axis xyz="0 0 1"/>
       <limit
@@ -68,5 +69,5 @@
       />
     </joint>
-    <link name="link_2">
+    <link name="${tf_prefix}link_2">
       <inertial>
         <origin rpy="0 0 0" xyz="0.064818 -0.11189 -0.038671"/>
@@ -90,8 +91,8 @@
       </collision>
     </link>
-    <joint name="joint_2" type="revolute">
+    <joint name="${tf_prefix}joint_2" type="revolute">
       <origin rpy="1.5708 0 -1.5708" xyz="0 0.0642 -0.16977"/>
-      <parent link="link_1"/>
-      <child link="link_2"/>
+      <parent link="${tf_prefix}link_1"/>
+      <child link="${tf_prefix}link_2"/>
       <axis xyz="0 0 -1"/>
       <limit
@@ -102,5 +103,5 @@
       />
     </joint>
-    <link name="link_3">
+    <link name="${tf_prefix}link_3">
       <inertial>
         <origin rpy="0 0 0" xyz="-0.00029765 -0.023661 -0.0019125"/>
@@ -124,8 +125,8 @@
       </collision>
     </link>
-    <joint name="joint_3" type="revolute">
+    <joint name="${tf_prefix}joint_3" type="revolute">
       <origin rpy="0 0 3.1416" xyz="0 -0.305 0.007"/>
-      <parent link="link_2"/>
-      <child link="link_3"/>
+      <parent link="${tf_prefix}link_2"/>
+      <child link="${tf_prefix}link_3"/>
       <axis xyz="0 0 -1"/>
       <limit
@@ -136,5 +137,5 @@
       />
     </joint>
-    <link name="link_4">
+    <link name="${tf_prefix}link_4">
       <inertial>
         <origin rpy="0 0 0" xyz="-0.0016798 -0.00057319 -0.074404"/>
@@ -158,8 +159,8 @@
       </collision>
     </link>
-    <joint name="joint_4" type="revolute">
+    <joint name="${tf_prefix}joint_4" type="revolute">
       <origin rpy="1.5708 0 -1.5708" xyz="0 0 0.0"/>
-      <parent link="link_3"/>
-      <child link="link_4"/>
+      <parent link="${tf_prefix}link_3"/>
+      <child link="${tf_prefix}link_4"/>
       <axis xyz="0 0 -1"/>
       <limit
@@ -170,5 +171,5 @@
       />
     </joint>
-    <link name="link_5">
+    <link name="${tf_prefix}link_5">
       <inertial>
         <origin rpy="0 0 0" xyz="0.0015066 -1.3102E-05 -0.012585"/>
@@ -192,8 +193,8 @@
       </collision>
     </link>
-    <joint name="joint_5" type="revolute">
+    <joint name="${tf_prefix}joint_5" type="revolute">
       <origin rpy="${pi} 0 -1.5708" xyz="0 0 -0.22263"/>
-      <parent link="link_4"/>
-      <child link="link_5"/>
+      <parent link="${tf_prefix}link_4"/>
+      <child link="${tf_prefix}link_5"/>
       <axis xyz="1 0 0"/>
       <limit
@@ -204,5 +205,5 @@
       />
     </joint>
-    <link name="link_6">
+    <link name="${tf_prefix}link_6">
       <inertial>
         <origin rpy="0 0 0" xyz="2.9287E-10 -1.6472E-09 0.0091432"/>
@@ -226,8 +227,8 @@
       </collision>
     </link>
-    <joint name="joint_6" type="revolute">
+    <joint name="${tf_prefix}joint_6" type="revolute">
       <origin rpy="0 0 3.1416" xyz="0.000 0 ${robot_parameters['l6_length']}"/>
-      <parent link="link_5"/>
-      <child link="link_6"/>
+      <parent link="${tf_prefix}link_5"/>
+      <child link="${tf_prefix}link_6"/>
       <axis xyz="0 0 1"/>
       <limit
@@ -239,8 +240,8 @@
     </joint>
     <!-- center of the end effector mounting surface on link_6 -->
-    <link name="ee_link" />
-    <joint name="ee_joint" type="fixed">
-      <parent link="link_6" />
-      <child link="ee_link" />
+    <link name="${tf_prefix}ee_link" />
+    <joint name="${tf_prefix}ee_joint" type="fixed">
+      <parent link="${tf_prefix}link_6" />
+      <child link="${tf_prefix}ee_link" />
       <origin xyz="0 0 0.0" rpy="0 0 0" />
     </joint>

Commit message: Update ar_macro.xacro

File: annin_ar4_description/urdf/ar_macro.xacro (robot description, xacro)
@@ -1,249 +1,25 @@
-<?xml version="1.0" encoding="utf-8"?>
-<robot xmlns:xacro="http://wiki.ros.org/xacro">
-  <xacro:macro name="ar_robot" params="
-    tf_prefix
-    parent
-    *origin
-    robot_parameters_file
-  ">
-    <xacro:property name="robot_parameters" value="${xacro.load_yaml(robot_parameters_file)}"/>
-    <joint name="${tf_prefix}base_joint" type="fixed">
-      <xacro:insert_block name="origin" />
-      <parent link="${parent}"/>
-      <child link="${tf_prefix}base_link" />
-    </joint>
-    <link name="${tf_prefix}base_link">
-      <inertial>
-        <origin rpy="0 0 0" xyz="-4.6941E-06 0.054174 0.038824"/>
-        <mass value="0.7102"/>
-        <inertia ixx="0.0039943" ixy="3.697E-07" ixz="-5.7364E-08" iyy="0.0014946" iyz="-0.00036051" izz="0.0042554"/>
-      </inertial>
-      <visual>
-        <origin rpy="0 0 0" xyz="0 0 0"/>
-        <geometry>
-          <mesh filename="file://$(find annin_ar4_description)/meshes/${robot_parameters['mesh_dir']}/base_link.STL"/>
-        </geometry>
-        <material name="">
-          <color rgba="1 1 0 1"/>
-        </material>
-      </visual>
-      <collision>
-        <origin rpy="0 0 0" xyz="0 0 0"/>
-        <geometry>
-          <mesh filename="file://$(find annin_ar4_description)/meshes/${robot_parameters['mesh_dir']}/base_link.STL"/>
-        </geometry>
-      </collision>
-    </link>
-    <link name="${tf_prefix}link_1">
-      <inertial>
-        <origin rpy="0 0 0" xyz="-0.022706 0.04294 -0.12205"/>
-        <mass value="0.88065"/>
-        <inertia ixx="0.0034" ixy="0.00042296" ixz="-0.00089231" iyy="0.0041778" iyz="0.0010848" izz="0.0027077"/>
-      </inertial>
-      <visual>
-        <origin rpy="0 0 0" xyz="0 0 0"/>
-        <geometry>
-          <mesh filename="file://$(find annin_ar4_description)/meshes/${robot_parameters['mesh_dir']}/link_1.STL"/>
-        </geometry>
-        <material name="">
-          <color rgba="1 1 0 1"/>
-        </material>
-      </visual>
-      <collision>
-        <origin rpy="0 0 0" xyz="0 0 0"/>
-        <geometry>
-          <mesh filename="file://$(find annin_ar4_description)/meshes/${robot_parameters['mesh_dir']}/link_1.STL"/>
-        </geometry>
-      </collision>
-    </link>
-    <joint name="${tf_prefix}joint_1" type="revolute">
-      <origin rpy="${pi} 0 0" xyz="0 0 0"/>
-      <parent link="${tf_prefix}base_link"/>
-      <child link="${tf_prefix}link_1"/>
-      <axis xyz="0 0 1"/>
-      <limit
-        lower="${robot_parameters['j1_limit_min']}"
-        upper="${robot_parameters['j1_limit_max']}"
-        effort="-1"
-        velocity="1.0472"
-      />
-    </joint>
-    <link name="${tf_prefix}link_2">
-      <inertial>
-        <origin rpy="0 0 0" xyz="0.064818 -0.11189 -0.038671"/>
-        <mass value="0.57738"/>
-        <inertia ixx="0.0047312" ixy="0.0022624" ixz="0.00032144" iyy="0.0020836" iyz="-0.00056569" izz="0.0056129"/>
-      </inertial>
-      <visual>
-        <origin rpy="0 0 0" xyz="0 0 0"/>
-        <geometry>
-          <mesh filename="file://$(find annin_ar4_description)/meshes/${robot_parameters['mesh_dir']}/link_2.STL"/>
-        </geometry>
-        <material name="">
-          <color rgba="1 1 0 1"/>
-        </material>
-      </visual>
-      <collision>
-        <origin rpy="0 0 0" xyz="0 0 0"/>
-        <geometry>
-          <mesh filename="file://$(find annin_ar4_description)/meshes/${robot_parameters['mesh_dir']}/link_2.STL"/>
-        </geometry>
-      </collision>
-    </link>
-    <joint name="${tf_prefix}joint_2" type="revolute">
-      <origin rpy="1.5708 0 -1.5708" xyz="0 0.0642 -0.16977"/>
-      <parent link="${tf_prefix}link_1"/>
-      <child link="${tf_prefix}link_2"/>
-      <axis xyz="0 0 -1"/>
-      <limit
-        lower="${robot_parameters['j2_limit_min']}"
-        upper="${robot_parameters['j2_limit_max']}"
-        effort="-1"
-        velocity="1.0472"
-      />
-    </joint>
-    <link name="${tf_prefix}link_3">
-      <inertial>
-        <origin rpy="0 0 0" xyz="-0.00029765 -0.023661 -0.0019125"/>
-        <mass value="0.1787"/>
-        <inertia ixx="0.0001685" ixy="-2.7713E-05" ixz="5.6885E-06" iyy="0.00012865" iyz="2.9256E-05" izz="0.00020744"/>
-      </inertial>
-      <visual>
-        <origin rpy="0 0 0" xyz="0 0 0"/>
-        <geometry>
-          <mesh filename="file://$(find annin_ar4_description)/meshes/${robot_parameters['mesh_dir']}/link_3.STL"/>
-        </geometry>
-        <material name="">
-          <color rgba="1 1 0 1"/>
-        </material>
-      </visual>
-      <collision>
-        <origin rpy="0 0 0" xyz="0 0 0"/>
-        <geometry>
-          <mesh filename="file://$(find annin_ar4_description)/meshes/${robot_parameters['mesh_dir']}/link_3.STL"/>
-        </geometry>
-      </collision>
-    </link>
-    <joint name="${tf_prefix}joint_3" type="revolute">
-      <origin rpy="0 0 3.1416" xyz="0 -0.305 0.007"/>
-      <parent link="${tf_prefix}link_2"/>
-      <child link="${tf_prefix}link_3"/>
-      <axis xyz="0 0 -1"/>
-      <limit
-        lower="${robot_parameters['j3_limit_min']}"
-        upper="${robot_parameters['j3_limit_max']}"
-        effort="-1"
-        velocity="1.0472"
-      />
-    </joint>
-    <link name="${tf_prefix}link_4">
-      <inertial>
-        <origin rpy="0 0 0" xyz="-0.0016798 -0.00057319 -0.074404"/>
-        <mass value="0.34936"/>
-        <inertia ixx="0.0030532" ixy="-1.8615E-05" ixz="-7.0047E-05" iyy="0.0031033" iyz="-2.3301E-05" izz="0.00022264"/>
-      </inertial>
-      <visual>
-        <origin rpy="0 0 0" xyz="0 0 0"/>
-        <geometry>
-          <mesh filename="file://$(find annin_ar4_description)/meshes/${robot_parameters['mesh_dir']}/link_4.STL"/>
-        </geometry>
-        <material name="">
-          <color rgba="1 1 0 1"/>
-        </material>
-      </visual>
-      <collision>
-        <origin rpy="0 0 0" xyz="0 0 0"/>
-        <geometry>
-          <mesh filename="file://$(find annin_ar4_description)/meshes/${robot_parameters['mesh_dir']}/link_4.STL"/>
-        </geometry>
-      </collision>
-    </link>
-    <joint name="${tf_prefix}joint_4" type="revolute">
-      <origin rpy="1.5708 0 -1.5708" xyz="0 0 0.0"/>
-      <parent link="${tf_prefix}link_3"/>
-      <child link="${tf_prefix}link_4"/>
-      <axis xyz="0 0 -1"/>
-      <limit
-        lower="${robot_parameters['j4_limit_min']}"
-        upper="${robot_parameters['j4_limit_max']}"
-        effort="-1"
-        velocity="1.0472"
-      />
-    </joint>
-    <link name="${tf_prefix}link_5">
-      <inertial>
-        <origin rpy="0 0 0" xyz="0.0015066 -1.3102E-05 -0.012585"/>
-        <mass value="0.11562"/>
-        <inertia ixx="5.5035E-05" ixy="-1.019E-08" ixz="-2.6243E-06" iyy="8.2921E-05" iyz="1.4437E-08" izz="5.2518E-05"/>
-      </inertial>
-      <visual>
-        <origin rpy="0 0 0" xyz="0 0 0"/>
-        <geometry>
-          <mesh filename="file://$(find annin_ar4_description)/meshes/${robot_parameters['mesh_dir']}/link_5.STL"/>
-        </geometry>
-        <material name="">
-          <color rgba="1 1 0 1"/>
-        </material>
-      </visual>
-      <collision>
-        <origin rpy="0 0 0" xyz="0 0 0"/>
-        <geometry>
-          <mesh filename="file://$(find annin_ar4_description)/meshes/${robot_parameters['mesh_dir']}/link_5.STL"/>
-        </geometry>
-      </collision>
-    </link>
-    <joint name="${tf_prefix}joint_5" type="revolute">
-      <origin rpy="${pi} 0 -1.5708" xyz="0 0 -0.22263"/>
-      <parent link="${tf_prefix}link_4"/>
-      <child link="${tf_prefix}link_5"/>
-      <axis xyz="1 0 0"/>
-      <limit
-        lower="${robot_parameters['j5_limit_min']}"
-        upper="${robot_parameters['j5_limit_max']}"
-        effort="-1"
-        velocity="1.0472"
-      />
-    </joint>
-    <link name="${tf_prefix}link_6">
-      <inertial>
-        <origin rpy="0 0 0" xyz="2.9287E-10 -1.6472E-09 0.0091432"/>
-        <mass value="0.013863"/>
-        <inertia ixx="1.3596E-06" ixy="3.0585E-13" ixz="5.7102E-14" iyy="1.7157E-06" iyz="6.3369E-09" izz="2.4332E-06"/>
-      </inertial>
-      <visual>
-        <origin rpy="0 0 0" xyz="0 0 0"/>
-        <geometry>
-          <mesh filename="file://$(find annin_ar4_description)/meshes/${robot_parameters['mesh_dir']}/link_6.STL"/>
-        </geometry>
-        <material name="">
-          <color rgba="1 1 0 1"/>
-        </material>
-      </visual>
-      <collision>
-        <origin rpy="0 0 0" xyz="0 0 0"/>
-        <geometry>
-          <mesh filename="file://$(find annin_ar4_description)/meshes/${robot_parameters['mesh_dir']}/link_6.STL"/>
-        </geometry>
-      </collision>
-    </link>
-    <joint name="${tf_prefix}joint_6" type="revolute">
-      <origin rpy="0 0 3.1416" xyz="0.000 0 ${robot_parameters['l6_length']}"/>
-      <parent link="${tf_prefix}link_5"/>
-      <child link="${tf_prefix}link_6"/>
-      <axis xyz="0 0 1"/>
-      <limit
-        lower="${robot_parameters['j6_limit_min']}"
-        upper="${robot_parameters['j6_limit_max']}"
-        effort="-1"
-        velocity="1.0472"
-      />
-    </joint>
-    <!-- center of the end effector mounting surface on link_6 -->
-    <link name="${tf_prefix}ee_link" />
-    <joint name="${tf_prefix}ee_joint" type="fixed">
-      <parent link="${tf_prefix}link_6" />
-      <child link="${tf_prefix}ee_link" />
-      <origin xyz="0 0 0.0" rpy="0 0 0" />
-    </joint>
-  </xacro:macro>
+<?xml version="1.0"?>
+<robot xmlns:xacro="http://wiki.ros.org/xacro" name="$(arg ar_model)">
+  <xacro:arg name="tf_prefix" default="" />
+  <xacro:arg name="include_gripper" default="false"/>
+  <xacro:arg name="include_spraygun" default="true"/> <!--← 全角スペースを削除 -->
+  <xacro:include filename="$(find annin_ar4_description)/urdf/ar_macro.xacro"/>
+  <link name="world" />
+  <xacro:ar_robot
+    tf_prefix="$(arg tf_prefix)"
+    parent="world"
+    robot_parameters_file="$(find annin_ar4_description)/config/$(arg ar_model).yaml"
+  >
+    <origin xyz="0 0 0" rpy="0 0 0" />
+  </xacro:ar_robot>
+  <!-- グリッパーを追加 -->
+  <xacro:if value="$(arg include_gripper)">
+    <xacro:include filename="$(find annin_ar4_description)/urdf/ar_gripper_macro.xacro"/>
+    <xacro:ar_gripper parent="${tf_prefix}ee_link" /> <!-- tf_prefixを適用 -->
+  </xacro:if>
+  <!-- スプレーガンを追加 -->
+  <xacro:if value="$(arg include_spraygun)">
+    <xacro:include filename="$(find annin_ar4_description)/urdf/ar_spraygun_macro.xacro"/>
+    <xacro:ar_spraygun parent="${tf_prefix}ee_link" /> <!-- tf_prefixを適用 -->
+  </xacro:if>
 </robot>
