Commit message: Update and rename ar_spraygun_macro to ar_spraygun_macro.xacro

File: annin_ar4_description/urdf/ar_spraygun_macro.xacro (robot description, xacro)
@@ -3,5 +3,5 @@
     <visual>
       <geometry>
-        <mesh filename="package://your_package/meshes/gripper.stl"/>
+         <mesh filename="file://$(find annin_ar4_description)/meshes/ar4_gripper/gripper_base_link.stl" />
       </geometry>
     </visual>

Commit message: Update ar_spraygun_macro.xacro

File: annin_ar4_description/urdf/ar_spraygun_macro.xacro (robot description, xacro)
@@ -3,5 +3,5 @@
     <visual>
       <geometry>
-         <mesh filename="file://$(find annin_ar4_description)/meshes/ar4_gripper/gripper_base_link.stl" />
+         <mesh filename="file://$(find annin_ar4_description)/meshes/ar4_mk3/土台_V5 v4.stl" />
       </geometry>
     </visual>

Commit message: Update ar_spraygun_macro.xacro

File: annin_ar4_description/urdf/ar_spraygun_macro.xacro (robot description, xacro)
@@ -8,5 +8,5 @@
     <collision>
       <geometry>
-        <mesh filename="package://your_package/meshes/gripper.stl"/>
+       <mesh filename="file://$(find annin_ar4_description)/meshes/ar4_mk3/土台_V5 v4.stl" />
       </geometry>
     </collision>

Commit message: Update ar_spraygun_macro.xacro

File: annin_ar4_description/urdf/ar_spraygun_macro.xacro (robot description, xacro)
@@ -1,13 +1,22 @@
-<!-- 新しいリンク -->
+<?xml version="1.0"?>
+<robot xmlns:xacro="http://wiki.ros.org/xacro">
+  <!-- スプレーガンのリンク -->
   <link name="spray_link">
     <visual>
       <geometry>
-         <mesh filename="file://$(find annin_ar4_description)/meshes/ar4_mk3/土台_V5 v4.stl" />
+        <mesh filename="file://$(find annin_ar4_description)/meshes/ar4_mk3/土台_V5 v4.stl" />
       </geometry>
     </visual>
     <collision>
       <geometry>
-       <mesh filename="file://$(find annin_ar4_description)/meshes/ar4_mk3/土台_V5 v4.stl" />
+        <mesh filename="file://$(find annin_ar4_description)/meshes/ar4_mk3/土台_V5 v4.stl" />
       </geometry>
     </collision>
   </link>
+  <!-- `ee_link` と `spray_link` を接続 -->
+  <joint name="spray_joint" type="fixed">
+    <parent link="ee_link"/>
+    <child link="spray_link"/>
+    <origin xyz="0 0 0" rpy="0 0 0"/> <!-- 必要に応じて調整 -->
+  </joint>
+</robot>

Commit message: Update ar_spraygun_macro.xacro

File: annin_ar4_description/urdf/ar_spraygun_macro.xacro (robot description, xacro)
@@ -5,10 +5,10 @@
     <visual>
       <geometry>
-        <mesh filename="file://$(find annin_ar4_description)/meshes/ar4_mk3/土台_V5 v4.stl" />
+        <mesh filename="file://$(find annin_ar4_description)/meshes/ar4_mk3/spraygun_EE.stl" />
       </geometry>
     </visual>
     <collision>
       <geometry>
-        <mesh filename="file://$(find annin_ar4_description)/meshes/ar4_mk3/土台_V5 v4.stl" />
+        <mesh filename="file://$(find annin_ar4_description)/meshes/ar4_mk3/spraygun_EE.stl" />
       </geometry>
     </collision>

Commit message: Update ar_spraygun_macro.xacro

File: annin_ar4_description/urdf/ar_spraygun_macro.xacro (robot description, xacro)
@@ -1,22 +1,19 @@
-<?xml version="1.0"?>
-<robot xmlns:xacro="http://wiki.ros.org/xacro">
-  <!-- スプレーガンのリンク -->
+<xacro:macro name="ar_spraygun" params="parent">
+  <joint name="spray_joint" type="fixed">
+    <parent link="${parent}"/>
+    <child link="spray_link"/>
+    <origin xyz="0 0 0" rpy="0 0 0"/>
+  </joint>
   <link name="spray_link">
     <visual>
       <geometry>
-        <mesh filename="file://$(find annin_ar4_description)/meshes/ar4_mk3/spraygun_EE.stl" />
+        <mesh filename="file://$(find annin_ar4_description)/meshes/ar4_mk3/spraygun_EE.stl"/>
       </geometry>
     </visual>
     <collision>
       <geometry>
-        <mesh filename="file://$(find annin_ar4_description)/meshes/ar4_mk3/spraygun_EE.stl" />
+        <mesh filename="file://$(find annin_ar4_description)/meshes/ar4_mk3/spraygun_EE.stl"/>
       </geometry>
     </collision>
   </link>
-  <!-- `ee_link` と `spray_link` を接続 -->
-  <joint name="spray_joint" type="fixed">
-    <parent link="ee_link"/>
-    <child link="spray_link"/>
-    <origin xyz="0 0 0" rpy="0 0 0"/> <!-- 必要に応じて調整 -->
-  </joint>
-</robot>
+</xacro:macro>

Commit message: Update ar_spraygun_macro.xacro

File: annin_ar4_description/urdf/ar_spraygun_macro.xacro (robot description, xacro)
@@ -1,21 +1,21 @@
-<?xml version="1.0" encoding="utf-8"?>
+<?xml version="1.0"?>
 <robot xmlns:xacro="http://wiki.ros.org/xacro">
-<xacro:macro name="ar_spraygun" params="parent">
-  <joint name="spray_joint" type="fixed">
-    <parent link="${parent}"/>
-    <child link="spray_link"/>
-    <origin xyz="0 0 0" rpy="0 0 0"/>
-  </joint>
-  <link name="spray_link">
-    <visual>
-      <geometry>
-        <mesh filename="file://$(find annin_ar4_description)/meshes/ar4_mk3/spraygun_EE.stl"/>
-      </geometry>
-    </visual>
-    <collision>
-      <geometry>
-        <mesh filename="file://$(find annin_ar4_description)/meshes/ar4_mk3/spraygun_EE.stl"/>
-      </geometry>
-    </collision>
-  </link>
-</xacro:macro>
+  <xacro:macro name="ar_spraygun" params="parent">
+    <link name="spraygun_link">
+      <visual>
+        <origin rpy="0 0 0" xyz="0 0 0.1"/>
+        <geometry>
+          <mesh filename="file://$(find annin_ar4_description)/meshes/ar4_mk3/spraygun_EE.stl"/>
+        </geometry>
+        <material name="">
+          <color rgba="0.5 0.5 0.5 1"/>
+        </material>
+      </visual>
+    </link>
+    <joint name="spraygun_joint" type="fixed">
+      <parent link="${parent}" />
+      <child link="spraygun_link" />
+      <origin xyz="0 0 0.1" rpy="0 0 0"/>
+    </joint>
+  </xacro:macro>
+</robot>

Commit message: Update ar_spraygun_macro.xacro

File: annin_ar4_description/urdf/ar_spraygun_macro.xacro (robot description, xacro)
@@ -16,5 +16,5 @@
       <parent link="${parent}" />
       <child link="spraygun_link" />
-      <origin xyz="0 0 0.1" rpy="0 0 0"/>
+      <origin xyz="0 0 0.0" rpy="0 0 0"/>
     </joint>
   </xacro:macro>

Commit message: Update ar_spraygun_macro.xacro

File: annin_ar4_description/urdf/ar_spraygun_macro.xacro (robot description, xacro)
@@ -1,5 +1,5 @@
 <?xml version="1.0"?>
 <robot xmlns:xacro="http://wiki.ros.org/xacro">
-  <xacro:macro name="ar_spraygun" params="parent">
+  <xacro:macro name="ar_spraygun" params="ee_link">
     <link name="spraygun_link">
       <visual>
@@ -14,5 +14,5 @@
     </link>
     <joint name="spraygun_joint" type="fixed">
-      <parent link="${parent}" />
+      <parent link="${ee_link}" />
       <child link="spraygun_link" />
       <origin xyz="0 0 0.0" rpy="0 0 0"/>

Commit message: Update ar_spraygun_macro.xacro

File: annin_ar4_description/urdf/ar_spraygun_macro.xacro (robot description, xacro)
@@ -1,5 +1,5 @@
 <?xml version="1.0"?>
 <robot xmlns:xacro="http://wiki.ros.org/xacro">
-  <xacro:macro name="ar_spraygun" params="ee_link">
+  <xacro:macro name="ar_spraygun" params="parent">
     <link name="spraygun_link">
       <visual>
@@ -14,5 +14,5 @@
     </link>
     <joint name="spraygun_joint" type="fixed">
-      <parent link="${ee_link}" />
+      <parent link="${parent}" />
       <child link="spraygun_link" />
       <origin xyz="0 0 0.0" rpy="0 0 0"/>

Commit message: Update ar_spraygun_macro.xacro

File: annin_ar4_description/urdf/ar_spraygun_macro.xacro (robot description, xacro)
@@ -1,6 +1,6 @@
 <?xml version="1.0"?>
 <robot xmlns:xacro="http://wiki.ros.org/xacro">
-  <xacro:macro name="ar_spraygun" params="parent">
-    <link name="spraygun_link">
+  <xacro:macro name="ar_spraygun" params="parent tf_prefix">
+    <link name="${tf_prefix}spraygun_link">
       <visual>
         <origin rpy="0 0 0" xyz="0 0 0.1"/>
@@ -13,7 +13,7 @@
       </visual>
     </link>
-    <joint name="spraygun_joint" type="fixed">
+    <joint name="${tf_prefix}spraygun_joint" type="fixed">
       <parent link="${parent}" />
-      <child link="spraygun_link" />
+      <child link="${tf_prefix}spraygun_link" />
       <origin xyz="0 0 0.0" rpy="0 0 0"/>
     </joint>

Commit message: Update ar_spraygun_macro.xacro

File: annin_ar4_description/urdf/ar_spraygun_macro.xacro (robot description, xacro)
@@ -14,7 +14,7 @@
     </link>
     <joint name="${tf_prefix}spraygun_joint" type="fixed">
-      <parent link="${parent}" />
-      <child link="${tf_prefix}spraygun_link" />
-      <origin xyz="0 0 0.0" rpy="0 0 0"/>
+     <parent link="${tf_prefix}${parent}" /> <!-- tf_prefixを適用 -->
+     <child link="${tf_prefix}spraygun_link" />
+     <origin xyz="0 0 0.0" rpy="0 0 0"/>
     </joint>
   </xacro:macro>

Commit message: Update ar_spraygun_macro.xacro

File: annin_ar4_description/urdf/ar_spraygun_macro.xacro (robot description, xacro)
@@ -14,5 +14,5 @@
     </link>
     <joint name="${tf_prefix}spraygun_joint" type="fixed">
-     <parent link="${tf_prefix}${parent}" /> <!-- tf_prefixを適用 -->
+     <parent link="${parent}" />
      <child link="${tf_prefix}spraygun_link" />
      <origin xyz="0 0 0.0" rpy="0 0 0"/>

Commit message: Update ar_spraygun_macro.xacro

File: annin_ar4_description/urdf/ar_spraygun_macro.xacro (robot description, xacro)
@@ -1,5 +1,5 @@
 <?xml version="1.0"?>
 <robot xmlns:xacro="http://wiki.ros.org/xacro">
-  <xacro:macro name="ar_spraygun" params="parent tf_prefix">
+　<xacro:macro name="ar_spraygun" params="parent tf_prefix">
     <link name="${tf_prefix}spraygun_link">
       <visual>

Commit message: Update ar_spraygun_macro.xacro

File: annin_ar4_description/urdf/ar_spraygun_macro.xacro (robot description, xacro)
@@ -1,5 +1,5 @@
 <?xml version="1.0"?>
 <robot xmlns:xacro="http://wiki.ros.org/xacro">
-　<xacro:macro name="ar_spraygun" params="parent tf_prefix">
+　<xacro:macro name="ar_spraygun" params="parent tf_prefix:=''" >
     <link name="${tf_prefix}spraygun_link">
       <visual>
