Commit message: Update ar_gripper_macro.xacro

File: annin_ar4_description/urdf/ar_gripper_macro.xacro (robot description, xacro)
@@ -1,11 +1,14 @@
 <?xml version="1.0" encoding="utf-8"?>
 <robot xmlns:xacro="http://wiki.ros.org/xacro">
-  <xacro:macro name="ar_gripper" params="parent">
-    <joint name="gripper_base_joint" type="fixed">
+  <xacro:macro name="ar_gripper" params="
+    tf_prefix
+    parent
+  ">
+    <joint name="${tf_prefix}gripper_base_joint" type="fixed">
       <origin xyz="0.0 0.0 0.0" rpy="-1.5708 0.0 0.0"/>
       <parent link="${parent}"/>
-      <child link="gripper_base_link"/>
+      <child link="${tf_prefix}gripper_base_link"/>
     </joint>
-    <link name="gripper_base_link">
+    <link name="${tf_prefix}gripper_base_link">
       <visual>
         <geometry>
@@ -27,5 +30,5 @@
       </inertial>
     </link>
-    <link name="gripper_jaw1_link">
+    <link name="${tf_prefix}gripper_jaw1_link">
       <visual>
         <geometry>
@@ -47,5 +50,5 @@
       </inertial>
     </link>
-    <link name="gripper_jaw2_link">
+    <link name="${tf_prefix}gripper_jaw2_link">
       <visual>
         <geometry>
@@ -67,18 +70,18 @@
       </inertial>
     </link>
-    <joint name="gripper_jaw1_joint" type="prismatic">
+    <joint name="${tf_prefix}gripper_jaw1_joint" type="prismatic">
       <origin xyz="0.0 -0.036 0" rpy="0.0 0.0 0.0"/>
-      <parent link="gripper_base_link"/>
-      <child link="gripper_jaw1_link"/>
-      <axis xyz="1 0 0"/>
-      <limit lower="-0.014" upper="0" effort="-1" velocity="1.0"/>
+      <parent link="${tf_prefix}gripper_base_link"/>
+      <child link="${tf_prefix}gripper_jaw1_link"/>
+      <axis xyz="-1 0 0"/>
+      <limit lower="0" upper="0.014" effort="-1" velocity="1.0"/>
     </joint>
-    <joint name="gripper_jaw2_joint" type="prismatic">
+    <joint name="${tf_prefix}gripper_jaw2_joint" type="prismatic">
       <origin xyz="0.0 -0.036 0" rpy="0.0 ${-pi} 0.0"/>
-      <parent link="gripper_base_link"/>
-      <child link="gripper_jaw2_link"/>
-      <axis xyz="1 0 0"/>
-      <limit lower="-0.014" upper="0" effort="-1" velocity="1.0"/>
-      <mimic joint="gripper_jaw1_joint" multiplier="1" offset="0"/>
+      <parent link="${tf_prefix}gripper_base_link"/>
+      <child link="${tf_prefix}gripper_jaw2_link"/>
+      <axis xyz="-1 0 0"/>
+      <limit lower="0" upper="0.014" effort="1000" velocity="1.0"/>
+      <mimic joint="${tf_prefix}gripper_jaw1_joint" multiplier="1" offset="0"/>
     </joint>
   </xacro:macro>
