Commit message: Update ar.ros2_control.xacro

File: annin_ar4_description/urdf/ar.ros2_control.xacro (robot description, xacro)
@@ -9,4 +9,5 @@
     joint_offset_parameters_file
     driver_parameters_file
+    tf_prefix
   ">
     <xacro:property name="robot_parameters"
@@ -22,7 +23,9 @@
         <param name="serial_port">${serial_port}</param>
         <param name="calibrate">${calibrate}</param>
+        <param name="calib_sequence">${driver_parameters['calib_sequence']}</param>
         <param name="velocity_control_enabled">${driver_parameters['velocity_control_enabled']}</param>
+        <param name="tf_prefix">${tf_prefix}</param>
       </hardware>
-      <joint name="joint_1">
+      <joint name="${tf_prefix}joint_1">
         <command_interface name="position">
           <param name="min">${robot_parameters['j1_limit_min']}</param>
@@ -38,5 +41,5 @@
         <param name="position_offset">${joint_offset_parameters['joint_1']}</param>
       </joint>
-      <joint name="joint_2">
+      <joint name="${tf_prefix}joint_2">
         <command_interface name="position">
           <param name="min">${robot_parameters['j2_limit_min']}</param>
@@ -52,5 +55,5 @@
         <param name="position_offset">${joint_offset_parameters['joint_2']}</param>
       </joint>
-      <joint name="joint_3">
+      <joint name="${tf_prefix}joint_3">
         <command_interface name="position">
           <param name="min">${robot_parameters['j3_limit_min']}</param>
@@ -66,5 +69,5 @@
         <param name="position_offset">${joint_offset_parameters['joint_3']}</param>
       </joint>
-      <joint name="joint_4">
+      <joint name="${tf_prefix}joint_4">
         <command_interface name="position">
           <param name="min">${robot_parameters['j4_limit_min']}</param>
@@ -80,5 +83,5 @@
         <param name="position_offset">${joint_offset_parameters['joint_4']}</param>
       </joint>
-      <joint name="joint_5">
+      <joint name="${tf_prefix}joint_5">
         <command_interface name="position">
           <param name="min">${robot_parameters['j5_limit_min']}</param>
@@ -94,5 +97,5 @@
         <param name="position_offset">${joint_offset_parameters['joint_5']}</param>
       </joint>
-      <joint name="joint_6">
+      <joint name="${tf_prefix}joint_6">
         <command_interface name="position">
           <param name="min">${robot_parameters['j6_limit_min']}</param>
